File: EDA files/EEZ DIB DCM224 r3B3.brd (EAGLE design)
At the start: 155 x 95 mm, 250 parts, among them IC1 Si8662AB-B-IS1, IC10 LT3763EFE#PBF, IC11 MC33274ADR2G, IC12 LT3763EFE#PBF, IC2 TPS54060DGQ, IC3 Si8641AB-B-IS1, IC4 M24C32-WMN6P, IC5 LP2985-33DBVR, IC6 74HC2G04GW,125, IC7 STM32F373C8T6, IC8 TL431B, IC9 MC33272ADR2G, J1 4907, J2 571-0500, J3 571-0100, J4 571-0500, J5 571-0100, Q1 BSP716NH6327XTSA1, Q10 NTD5867NLT4G, Q11 BSS205NH6327XTSA1, Q12 BSS84, Q2 NTD5867NLT4G, Q3 NTD5867NLT4G, Q4 NTD5867NLT4G, Q5 BSS205NH6327XTSA1, Q6 BSS84, Q7 BSP716NH6327XTSA1, Q8 NTD5867NLT4G, Q9 NTD5867NLT4G, X1 39-30-1020, X2 77317-104-28LF, X3 N.C., X4 DS1024-2*5R0, Y1 LF XTAL026392

Commit message: licenses logo, mechanical
Parts:
- removed U$3: (no value), logo:CE_5MM
- added FM3: FIDUCIAL_2, EEZ_Lib1:FIDUCIAL_DUAL
- C1: value 10n/200V -> 1u/100V
- moved C31 6.51 mm to (118.7, 53.1), turned to 0 degrees
- moved C30 2.43 mm to (122.0, 53.1), turned to 180 degrees
- moved Y1 1.65 mm to (120.0, 58.5)
- moved FM1 0.50 mm to (15.0, 92.5)
Connections:
- net GND: no longer Y1.2, Y1.4
Routing:
- net GND: track 117.8 -> 140.7 mm, vias 209 -> 207
- net OE#1: track 137.5 -> 141.2 mm
- net RCC_OSC_IN: track 9.06 -> 7.94 mm
- net CC_LED#1: track 107.1 -> 106.1 mm
- net RCC_OSC_OUT: track 16.3 -> 15.4 mm
- net VREF2: track 80.6 -> 79.8 mm
- net TEMP#1: track 47.9 -> 48.5 mm
Other:
- board text added: "+VAUX 2 NRESET 4 SYNC 6 SSDA 8 IRQ 10 CSB 12 MISO 14 GND 16 A2 18 GND 20 +12V 22 +5V 24 BOOT 26 UART_TX 28"
- board text added: "1 +3V3 3 NFAULT 5 SSCL 7 GND 9 CSA 11 GND 13 SCLK 15 MOSI 17 A0 19 A1 21 +12V 23 +5V 25 GND 27 UART_RX"
- board text added: "DIB (bottom view)"
- board text added: "EEZ DIB DCM224 (11/2020 r3B3)"
- board text added: "EEZ DIB DCM224 (11/2020 r3B3) Project source code: github.com/eez-open"
- board text removed: "EEZ DIB DCM224 (08/2020 r3B3)"
- board text removed: "EEZ DIB DCM224 (08/2020 r3B3) Project source code: github.com/eez-open"
