File: EDA files/EEZ DIB DCM224 r3B4.brd (EAGLE design)
At the start: 155 x 95 mm, 250 parts, among them IC1 Si8662AB-B-IS1, IC10 LT3763EFE#PBF, IC11 MC33274ADR2G, IC12 LT3763EFE#PBF, IC2 TPS54060DGQ, IC3 Si8641AB-B-IS1, IC4 M24C32-WMN6P, IC5 LP2985-33DBVR, IC6 74HC2G04GW,125, IC7 STM32F373C8T6, IC8 TL431B, IC9 MC33272ADR2G, J1 4907, J2 571-0500, J3 571-0100, J4 571-0500, J5 571-0100, Q1 BSP716NH6327XTSA1, Q10 NTD5867NLT4G, Q11 BSS205NH6327XTSA1, Q12 BSS84, Q2 NTD5867NLT4G, Q3 NTD5867NLT4G, Q4 NTD5867NLT4G, Q5 BSS205NH6327XTSA1, Q6 BSS84, Q7 BSP716NH6327XTSA1, Q8 NTD5867NLT4G, Q9 NTD5867NLT4G, X1 39-30-1020, X2 77317-104-28LF, X3 N.C., X4 DS1024-2*5R0, Y1 LF XTAL026392

Commit message: #1
Parts:
- added U$3: (no value), logo:CE_5MM
- OE#1, OE#2: value JP2-NOCUT -> JP2-NOCUT-0805; device EEZ_Lib1:JP2-NOCUT -> EEZ_Lib1:JP2-0805-NOCUT
- moved OE#1 0.25 mm to (126.4, 54.7)
Connections:
- net +3V3: no longer C34.2
- net GND: now also C34.2, R45.1, R68.1
- net VOUT1-: no longer R45.1
- net VOUT2-: no longer R68.1
Routing:
- net VOUT1-: track 130.5 -> 102.8 mm, vias 11 -> 10
- net VOUT2-: track 90.9 -> 63.6 mm, vias 11 -> 10
- net GND: track 140.7 -> 145.3 mm, vias 207 -> 209
- net +3V3: track 234.9 -> 233.8 mm, vias 17 -> 16
Other:
- board text added: "CH1"
- board text added: "CH2"
- board text added: "EEZ DIB DCM224 (07/2021 r3B4)"
- board text added: "EEZ DIB DCM224 (07/2021 r3B4) Project source code: github.com/eez-open"
- board text removed: "+VAUX 2 NRESET 4 SYNC 6 SSDA 8 IRQ 10 CSB 12 MISO 14 GND 16 A2 18 GND 20 +12V 22 +5V 24 BOOT 26 UART_TX 28"
- board text removed: "1 +3V3 3 NFAULT 5 SSCL 7 GND 9 CSA 11 GND 13 SCLK 15 MOSI 17 A0 19 A1 21 +12V 23 +5V 25 GND 27 UART_RX"
- board text removed: "DIB (bottom view)"
- board text removed: "EEZ DIB DCM224 (11/2020 r3B3)"
- board text removed: "EEZ DIB DCM224 (11/2020 r3B3) Project source code: github.com/eez-open"
