File: EDA files/EEZ DIB DCM224 r3B4.sch (EAGLE design)
At the start: 246 parts, among them IC1 Si8662AB-B-IS1, IC10 LT3763EFE#PBF, IC11 MC33274ADR2G, IC12 LT3763EFE#PBF, IC2 TPS54060DGQ, IC3 Si8641AB-B-IS1, IC4 M24C32-WMN6P, IC5 LP2985-33DBVR, IC6 74HC2G04GW,125, IC7 STM32F373C8T6, IC8 TL431B, IC9 MC33272ADR2G, J1 4907, J2 571-0500, J3 571-0100, J4 571-0500, J5 571-0100, Q1 BSP716NH6327XTSA1, Q10 NTD5867NLT4G, Q11 BSS205NH6327XTSA1, Q12 BSS84, Q2 NTD5867NLT4G, Q3 NTD5867NLT4G, Q4 NTD5867NLT4G, Q5 BSS205NH6327XTSA1, Q6 BSS84, Q7 BSP716NH6327XTSA1, Q8 NTD5867NLT4G, Q9 NTD5867NLT4G, X1 39-30-1020, X2 77317-104-28LF, X3 N.C., X4 DS1024-2*5R0, Y1 LF XTAL026392

Commit message: #1
Parts:
- OE#1, OE#2: value JP2-NOCUT -> JP2-NOCUT-0805; device EEZ_Lib1:JP2-NOCUT -> EEZ_Lib1:JP2-NOCUT-0805
Connections:
- net +3V3: no longer C34.2
- net GND: now also C34.2, R45.1, R68.1
- net VOUT1-: no longer R45.1
- net VOUT2-: no longer R68.1
Other:
- moved on the sheet: C34, R45, R68
